File: Avances/PCB/triatlon smd.kicad_pcb (KiCad board)
At the start: 2 copper layers, 68 x 54.3 mm, 8 parts, among them J2 BTS-1, J5 BTS-2, SW1 SW_DPST_x2

Commit message: triatlon smd.kicad_pcb
Routing:
- net +5V: track 133.3 -> 107.3 mm
Changed lines of the file:
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@@
 			(psa4output no)
 			(plot_black_and_white yes)
+			(plotinvisibletext no)
 			(sketchpadsonfab no)
 			(plotpadnumbers no)
@@
 			(net 8 "unconnected-(ESP32-3v3-Pad1)")
 			(pinfunction "3v3")
-			(pintype "input")
+			(pintype "input+no_connect")
 		)
 		(pad "2" thru_hole oval
@@
 			(net 19 "unconnected-(ESP32-EN{slash}RESET-Pad2)")
 			(pinfunction "EN/RESET")
-			(pintype "bidirectional")
+			(pintype "bidirectional+no_connect")
 		)
 		(pad "3" thru_hole oval
@@
 			(net 23 "unconnected-(ESP32-G36{slash}ADC0-Pad3)")
 			(pinfunction "G36/ADC0")
-			(pintype "bidirectional")
+			(pintype "bidirectional+no_connect")
 		)
 		(pad "4" thru_hole oval
@@
 			(net 10 "unconnected-(ESP32-G39{slash}ADC6-Pad4)")
 			(pinfunction "G39/ADC6")
-			(pintype "bidirectional")
+			(pintype "bidirectional+no_connect")
 		)
 		(pad "5" thru_hole oval
@@
 			(net 31 "unconnected-(ESP32-G34{slash}ADC15-Pad5)")
 			(pinfunction "G34/ADC15")
-			(pintype "bidirectional")
+			(pintype "bidirectional+no_connect")
 		)
 		(pad "6" thru_hole oval
@@
 			(net 26 "unconnected-(ESP32-G35{slash}ADC7-Pad6)")
 			(pinfunction "G35/ADC7")
-			(pintype "bidirectional")
+			(pintype "bidirectional+no_connect")
 		)
 		(pad "7" thru_hole oval
@@
 			(net 37 "unconnected-(ESP32-G32{slash}ADC4-Pad7)")
 			(pinfunction "G32/ADC4")
-			(pintype "bidirectional")
+			(pintype "bidirectional+no_connect")
 		)
 		(pad "8" thru_hole oval
@@
 			(net 18 "unconnected-(ESP32-G33{slash}ADC5-Pad8)")
 			(pinfunction "G33/ADC5")
-			(pintype "bidirectional")
+			(pintype "bidirectional+no_connect")
 		)
 		(pad "9" thru_hole oval
@@
 			(net 24 "unconnected-(ESP32-G25{slash}ADC18-Pad9)")
 			(pinfunction "G25/ADC18")
-			(pintype "bidirectional")
+			(pintype "bidirectional+no_connect")
 		)
 		(pad "10" thru_hole oval
@@
 			(net 12 "unconnected-(ESP32-G27{slash}ADC17-Pad11)")
 			(pinfunction "G27/ADC17")
-			(pintype "bidirectional")
+			(pintype "bidirectional+no_connect")
 		)
 		(pad "12" thru_hole oval
@@
 			(net 28 "unconnected-(ESP32-G14{slash}ADC16-Pad12)")
 			(pinfunction "G14/ADC16")
-			(pintype "bidirectional")
+			(pintype "bidirectional+no_connect")
 		)
 		(pad "13" thru_hole oval
@@
 			(net 36 "unconnected-(ESP32-G13{slash}ADC14-Pad15)")
 			(pinfunction "G13/ADC14")
-			(pintype "bidirectional")
+			(pintype "bidirectional+no_connect")
 		)
 		(pad "16" thru_hole oval
@@
 			(pintype "bidirectional+no_connect")
 		)
-		(pad "22" thru_hole oval
+		(pad "22" thru_hole circle
 			(at 10.16 20.95 270)
-			(size 3 1.8)
-			(drill 0.95)
+			(size 0.001 0.001)
+			(drill 0.0001)
 			(layers "*.Cu" "*.Mask")
 			(remove_unused_layers no)
@@
 			(pintype "bidirectional+no_connect")
 		)
-		(pad "23" thru_hole oval
+		(pad "23" thru_hole circle
 			(at 10.16 18.41 270)
-			(size 3 1.8)
-			(drill 0.95)
+			(size 0.001 0.001)
+			(drill 0.0001)
 			(layers "*.Cu" "*.Mask")
 			(remove_unused_layers no)
 			(net 15 "unconnected-(ESP32-G15{slash}ADC13-Pad23)")
 			(pinfunction "G15/ADC13")
-			(pintype "bidirectional")
+			(pintype "bidirectional+no_connect")
 		)
 		(pad "24" thru_hole oval
@@
 			(net 34 "unconnected-(ESP32-G2{slash}ADC12-Pad24)")
 			(pinfunction "G2/ADC12")
-			(pintype "bidirectional")
+			(pintype "bidirectional+no_connect")
 		)
 		(pad "25" thru_hole oval
@@
 			(net 25 "unconnected-(ESP32-G0{slash}ADC11-Pad25)")
 			(pinfunction "G0/ADC11")
-			(pintype "bidirectional")
+			(pintype "bidirectional+no_connect")
 		)
 		(pad "26" thru_hole oval
@@
 			(net 38 "unconnected-(ESP32-G17{slash}TX2-Pad28)")
 			(pinfunction "G17/TX2")
-			(pintype "bidirectional")
+			(pintype "bidirectional+no_connect")
 		)
 		(pad "29" thru_hole oval
@@
 			(net 32 "unconnected-(ESP32-G5-Pad29)")
 			(pinfunction "G5")
-			(pintype "bidirectional")
+			(pintype "bidirectional+no_connect")
 		)
 		(pad "30" thru_hole oval
@@
 			(net 30 "unconnected-(ESP32-G18-Pad30)")
 			(pinfunction "G18")
-			(pintype "bidirectional")
+			(pintype "bidirectional+no_connect")
 		)
 		(pad "31" thru_hole oval
@@
 			(net 27 "unconnected-(ESP32-G19-Pad31)")
 			(pinfunction "G19")
-			(pintype "bidirectional")
+			(pintype "bidirectional+no_connect")
 		)
 		(pad "32" thru_hole oval
@@
 			(net 16 "unconnected-(ESP32-G21-Pad33)")
 			(pinfunction "G21")
-			(pintype "bidirectional")
+			(pintype "bidirectional+no_connect")
 		)
 		(pad "34" thru_hole oval
@@
 	)
 	(segment
-		(start 39.63 42.91)
-		(end 39.62 42.92)
+		(start 75.38 78.79)
+		(end 85.69 78.79)
 		(width 1.5)
 		(layer "B.Cu")
@@
 	)
 	(segment
-		(start 49.87 76.07)
-		(end 49.87 71.91)
+		(start 49.07 78.44)
+		(end 49.87 77.64)
 		(width 1.5)
 		(layer "B.Cu")
@@
 	)
 	(segment
-		(start 83.48 52.29)
-		(end 88.66 57.47)
+		(start 49.07 78.79)
+		(end 49.07 78.44)
 		(width 1.5)
 		(layer "B.Cu")
@@
 	)
 	(segment
-		(start 39.62 42.92)
-		(end 48.99 52.29)
+		(start 51.02 78.79)
+		(end 75.38 78.79)
+		(width 1.5)
+		(layer "B.Cu")
+		(net 20)
+	)
+	(segment
+		(start 47.12 78.79)
+		(end 49.07 78.79)
+		(width 1.5)
+		(layer "B.Cu")
+		(net 20)
+	)
+	(segment
+		(start 75.29 71.91)
+		(end 75.29 78.7)
+		(width 1.5)
+		(layer "B.Cu")
+		(net 20)
+	)
+	(segment
+		(start 49.87 77.64)
+		(end 51.02 78.79)
+		(width 1.5)
+		(layer "B.Cu")
+		(net 20)
+	)
+	(segment
+		(start 45.9985 77.6685)
+		(end 47.12 78.79)
+		(width 1.5)
+		(layer "B.Cu")
+		(net 20)
+	)
+	(segment
+		(start 39.63 45.723)
+		(end 45.9985 52.0915)
+		(width 1.5)
+		(layer "B.Cu")
+		(net 20)
+	)
+	(segment
+		(start 85.69 78.79)
+		(end 91.68 72.8)
 		(width 1.5)
 		(layer "B.Cu")
@@
 	)
 	(segment
-		(start 88.66 57.47)
-		(end 88.66 65.96)
+		(start 49.87 71.91)
+		(end 49.87 77.64)
 		(width 1.5)
 		(layer "B.Cu")
@@
 	)
 	(segment
-		(start 75.29 71.91)
-		(end 75.29 78.52)
+		(start 45.9985 52.0915)
+		(end 45.9985 77.6685)
 		(width 1.5)
 		(layer "B.Cu")
@@
 	)
 	(segment
-		(start 91.68 68.98)
-		(end 91.68 72.8)
+		(start 39.63 42.91)
+		(end 39.63 45.723)
 		(width 1.5)
 		(layer "B.Cu")
@@
 	)
 	(segment
-		(start 52.53 78.73)
-		(end 49.87 76.07)
+		(start 75.29 78.7)
+		(end 75.38 78.79)
 		(width 1.5)
 		(layer "B.Cu")
@@
 	)
 	(segment
-		(start 85.75 78.73)
-		(end 52.53 78.73)
+		(start 39.63 42.91)
+		(end 39.62 42.92)
 		(width 1.5)
 		(layer "B.Cu")
@@
 	)
 	(segment
-		(start 88.66 65.96)
-		(end 91.68 68.98)
+		(start 51.02 78.79)
+		(end 49.07 78.79)
 		(width 1.5)
 		(layer "B.Cu")
-		(net 20)
-	)
-	(segment
-		(start 48.99 52.29)
-		(end 83.48 52.29)
-		(width 1.5)
-		(layer "B.Cu")
-		(net 20)
-	)
-	(segment
-		(start 91.68 72.8)
-		(end 85.75 78.73)
-		(width 1.5)
-		(layer "B.Cu")
